File: LapisHAT/LapisHAT.kicad_pcb (KiCad board)
At the start: 4 copper layers, 57 parts, among them J1 Conn_01x02, J10 Conn_01x02, J11 Conn_01x02, J12 Conn_01x02, J13 Conn_01x03, J14 Conn_01x03, J15 Conn_01x03, J16 Conn_01x03, J17 Conn_01x02, J18 Conn_01x02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

Commit message: pcb
Parts:
- removed C11, C12, C13, C14: 100u, Capacitor_SMD:CP_Elec_6.3x7.7
- removed C2: 330u, Capacitor_SMD:CP_Elec_4x5.4
- added G***: LOGO, EER_Logos:MI Logo Small, F.Cu at (114.3, 50.9)
- added G***: LOGO, EER_Logos:eer_logo_small, F.Cu at (91.2, 74.4)
- added G***: LOGO, EER_Logos:MUN Logo Small, F.Cu at (113.7, 67.2)
- added R10: 10k, Resistor_SMD:R_0603_1608Metric, F.Cu at (99.1, 66.7)
- added R11: 10k, Resistor_SMD:R_0603_1608Metric, F.Cu at (98.2, 55.0)
- C1: value 330u -> 120u; footprint Capacitor_SMD:CP_Elec_4x5.4 -> Capacitor_SMD:CP_Elec_10x12.6
- C3: footprint Capacitor_SMD:CP_Elec_10x12.5 -> Capacitor_SMD:CP_Elec_10x12.6
- C5, C8: footprint Capacitor_SMD:C_0805_2012Metric -> Capacitor_SMD:C_1206_3216Metric
- J17, J18, J5, J6: footprint footprints:Molex-43650-0227_-MFG -> Connector_Molex:Molex_Micro-Fit_3.0_43650-0200_1x02_P3.00mm_Horizontal
- J2: moved to B.Cu
- moved Q2 141.1 mm to (94.5, 91.2), turned to 180 degrees
- moved U4 139.1 mm to (98.1, 52.6), turned to 180 degrees
- moved U6 135.8 mm to (99.0, 64.6), turned to 180 degrees
- moved C1 126.9 mm to (111.0, 31.0)
- moved C4 125.7 mm to (94.6, 48.1), turned to 90 degrees
- moved C10 123.5 mm to (95.4, 60.2), turned to 90 degrees
- moved J18 122.0 mm to (83.6, 88.8), turned to 90 degrees
- moved J5 122.0 mm to (83.7, 56.4), turned to 90 degrees
- moved J17 121.9 mm to (83.6, 78.0), turned to 90 degrees
- moved J6 121.9 mm to (83.7, 67.2), turned to 90 degrees
- moved R2 119.7 mm to (98.3, 91.0), turned to 180 degrees
- moved C6 118.7 mm to (102.3, 49.6), turned to 90 degrees
- moved C9 116.5 mm to (101.6, 61.5), turned to 90 degrees
- moved C5 112.5 mm to (97.6, 47.6), turned to 90 degrees
- moved R1 112.3 mm to (98.3, 87.2), turned to 180 degrees
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Connections:
- net Net-(J17-Pin_2) renamed /Tooling/LED0_PIN
- net Net-(J18-Pin_2) renamed /Tooling/LED1_PIN
- J19 pad 14: /Pico/PI_SDA -> /Pico/PI_SCL
- J19 pad 15: /Pico/PI_SCL -> /Pico/PI_SDA
- J2 pad 10: unconnected-(J2-Pin_10-Pad10) -> GND
- J2 pad 13: unconnected-(J2-Pin_13-Pad13) -> GND
- J2 pad 19: unconnected-(J2-Pin_19-Pad19) -> GND
- J2 pad 26: unconnected-(J2-Pin_26-Pad26) -> GND
- J2 pad 29: unconnected-(J2-Pin_29-Pad29) -> GND
- J2 pad 3: unconnected-(J2-Pin_3-Pad3) -> +5V
- J2 pad 33: unconnected-(J2-Pin_33-Pad33) -> GND
- J2 pad 40: unconnected-(J2-Pin_40-Pad40) -> GND
- J4 pad 11: /Pico/ESC4 -> /Pico/ESC5
- J4 pad 12: /Pico/ESC5 -> /Pico/ESC4
- J5 pad 1: /Tooling/MOTOR0_OUT1 -> /Tooling/MOTOR0_OUT2
- J5 pad 2: /Tooling/MOTOR0_OUT2 -> /Tooling/MOTOR0_OUT1
- J6 pad 1: /Tooling/MOTOR1_OUT1 -> /Tooling/MOTOR1_OUT2
- J6 pad 2: /Tooling/MOTOR1_OUT2 -> /Tooling/MOTOR1_OUT1
- R12 pad 2: /Pico/PI_SDA -> /Pico/PI_SCL
- R13 pad 2: /Pico/PI_SCL -> /Pico/PI_SDA
- U4 pad 1: GND -> Net-(U4-IPROPI)
- U6 pad 1: GND -> Net-(U6-IPROPI)
Routing:
- net /Pico/PI_SDA: track 1.42 -> 42.3 mm, vias 1 -> 0
- net /Pico/PI_SCL: track 1.42 -> 37.1 mm, vias 1 -> 0
- net /Pico/MOTOR0_IN2: track 0.00 -> 33.8 mm
- net /Pico/MOTOR0_IN1: track 0.00 -> 32.2 mm
- net /Pico/ESC0: track 29.8 -> 56.2 mm
- net /Pico/MOTOR1_IN2: track 0.00 -> 25.8 mm
- net /Pico/SERVO3: track 0.00 -> 24.3 mm
- net /Pico/MOTOR1_IN1: track 0.00 -> 24.1 mm
- net /Pico/SERVO2: track 0.00 -> 20.3 mm
- net /Pico/ESC5: track 63.8 -> 43.7 mm
- net /Pico/ESC4: track 52.6 -> 34.7 mm
- net /Pico/ESC1: track 34.5 -> 49.0 mm
- net /Pico/SERVO1: track 0.00 -> 13.7 mm
- net /Pico/LED0: track 0.00 -> 13.4 mm
- net /Pico/LED1: track 0.00 -> 13.1 mm
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- added copper zone on F.Cu, net +12V
- added copper zone on In1.Cu, net +12V
- added copper zone on F.Cu, net +5V
- added copper zone on F.Cu, net /Tooling/LED0_PIN
- added copper zone on F.Cu, net /Tooling/LED1_PIN
- added copper zone on F.Cu, net /Tooling/MOTOR0_OUT1
- added copper zone on F.Cu, net /Tooling/MOTOR0_OUT2
- added copper zone on F.Cu, net /Tooling/MOTOR1_OUT1
- added copper zone on F.Cu, net /Tooling/MOTOR1_OUT2
Other:
- board outline added: 71.1 x 86.3 mm
- board text added: "Tooling Board Evan Whelan 2026"
