File: LapisHAT/pico.kicad_sch (KiCad schematic)
At the start: 16 parts, among them J1 Conn_01x02, J19 Conn_01x20, J2 Conn_02x20_Odd_Even, J4 Conn_01x20

Commit message: Move connectors and add correct 5v cap
Parts:
- C3: value 100u -> 120u; footprint Capacitor_SMD:CP_Elec_6.3x7.7 -> Capacitor_SMD:CP_Elec_10x12.5; LCSC C3338 -> C24725845
Connections:
- net ESC0: now also J4.6 (Pin_6); no longer J4.14 (Pin_14)
- net ESC1: now also J4.7 (Pin_7); no longer J4.15 (Pin_15)
- net ESC2: now also J4.9 (Pin_9); no longer J4.16 (Pin_16)
- net ESC3: now also J4.10 (Pin_10); no longer J4.17 (Pin_17)
- net ESC4: now also J4.11 (Pin_11); no longer J4.19 (Pin_19)
- net ESC5: now also J4.12 (Pin_12); no longer J4.20 (Pin_20)
- net LED0: now also J4.19 (Pin_19); no longer J4.11 (Pin_11)
- net LED1: now also J4.20 (Pin_20); no longer J4.12 (Pin_12)
- net MOTOR0_IN1: now also J4.14 (Pin_14); no longer J4.6 (Pin_6)
- net MOTOR0_IN2: now also J4.15 (Pin_15); no longer J4.7 (Pin_7)
- net MOTOR1_IN1: now also J4.16 (Pin_16); no longer J4.9 (Pin_9)
- net MOTOR1_IN2: now also J4.17 (Pin_17); no longer J4.10 (Pin_10)
Changed lines of the file:
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@@
+		)
+	)
+	(hierarchical_label "LED1"
+		(shape output)
+		(at 80.01 85.09 180)
+		(effects
+			(font
+				(size 1.27 1.27)
+			)
+			(justify right)
+		)
+	)
+	(hierarchical_label "ESC5"
+		(shape output)
+		(at 80.01 64.77 180)
+		(effects
+			(font
+				(size 1.27 1.27)
+			)
+			(justify right)
+		)
+	)
+	(hierarchical_label "SERVO2"
+		(shape output)
+		(at 124.46 77.47 0)
+		(effects
+			(font
+				(size 1.27 1.27)
+			)
+			(justify left)
+		)
+	)
+	(hierarchical_label "ESC0"
+		(shape output)
+		(at 80.01 49.53 180)
+		(effects
+			(font
+				(size 1.27 1.27)
+			)
+			(justify right)
+		)
+	)
+	(hierarchical_label "MOTOR0_IN2"
+		(shape output)
+		(at 80.01 72.39 180)
+		(effects
+			(font
+				(size 1.27 1.27)
+			)
+			(justify right)
+		)
+	)
+	(hierarchical_label "ESC1"
+		(shape output)
+		(at 80.01 52.07 180)
+		(effects
+			(font
+				(size 1.27 1.27)
+			)
+			(justify right)
+		)
+	)
+	(hierarchical_label "ESC2"
+		(shape output)
+		(at 80.01 57.15 180)
+		(effects
+			(font
+				(size 1.27 1.27)
+			)
+			(justify right)
 		)
 	)
 	(hierarchical_label "MOTOR1_IN1"
 		(shape output)
-		(at 80.01 57.15 180)
+		(at 80.01 74.93 180)
 		(effects
 			(font
@@
 	(hierarchical_label "ESC3"
 		(shape output)
+		(at 80.01 59.69 180)
+		(effects
+			(font
+				(size 1.27 1.27)
+			)
+			(justify right)
+		)
+	)
+	(hierarchical_label "MOTOR1_IN2"
+		(shape output)
 		(at 80.01 77.47 180)
 		(effects
@@
 		)
 	)
-	(hierarchical_label "SERVO2"
-		(shape output)
-		(at 124.46 77.47 0)
+	(hierarchical_label "LED0"
+		(shape output)
+		(at 80.01 82.55 180)
+		(effects
+			(font
+				(size 1.27 1.27)
+			)
+			(justify right)
+		)
+	)
+	(hierarchical_label "MOTOR0_IN1"
+		(shape output)
+		(at 80.01 69.85 180)
+		(effects
+			(font
+				(size 1.27 1.27)
+			)
+			(justify right)
+		)
+	)
+	(hierarchical_label "SERVO3"
+		(shape output)
+		(at 124.46 74.93 0)
 		(effects
 			(font
@@
 		)
 	)
-	(hierarchical_label "ESC2"
-		(shape output)
-		(at 80.01 74.93 180)
-		(effects
-			(font
-				(size 1.27 1.27)
-			)
-			(justify right)
-		)
-	)
 	(hierarchical_label "ESC4"
 		(shape output)
-		(at 80.01 82.55 180)
-		(effects
-			(font
-				(size 1.27 1.27)
-			)
-			(justify right)
-		)
-	)
-	(hierarchical_label "MOTOR0_IN2"
-		(shape output)
-		(at 80.01 52.07 180)
-		(effects
-			(font
-				(size 1.27 1.27)
-			)
-			(justify right)
-		)
-	)
-	(hierarchical_label "ESC0"
-		(shape output)
-		(at 80.01 69.85 180)
-		(effects
-			(font
-				(size 1.27 1.27)
-			)
-			(justify right)
-		)
-	)
-	(hierarchical_label "LED0"
-		(shape output)
 		(at 80.01 62.23 180)
 		(effects
@@
 		)
 	)
-	(hierarchical_label "SERVO3"
-		(shape output)
-		(at 124.46 74.93 0)
+	(hierarchical_label "SERVO0"
+		(shape output)
+		(at 124.46 85.09 0)
 		(effects
 			(font
@@
 		)
 	)
-	(hierarchical_label "MOTOR1_IN2"
-		(shape output)
-		(at 80.01 59.69 180)
-		(effects
-			(font
-				(size 1.27 1.27)
-			)
-			(justify right)
-		)
-	)
-	(hierarchical_label "SERVO0"
-		(shape output)
-		(at 124.46 85.09 0)
+	(hierarchical_label "SERVO1"
+		(shape output)
+		(at 124.46 82.55 0)
 		(effects
 			(font
@@
 			)
 			(justify left)
-		)
-	)
-	(hierarchical_label "SERVO1"
-		(shape output)
-		(at 124.46 82.55 0)
-		(effects
-			(font
-				(size 1.27 1.27)
-			)
-			(justify left)
-		)
-	)
-	(hierarchical_label "ESC5"
-		(shape output)
-		(at 80.01 85.09 180)
-		(effects
-			(font
-				(size 1.27 1.27)
-			)
-			(justify right)
-		)
-	)
-	(hierarchical_label "LED1"
-		(shape output)
-		(at 80.01 64.77 180)
-		(effects
-			(font
-				(size 1.27 1.27)
-			)
-			(justify right)
-		)
-	)
-	(hierarchical_label "ESC1"
-		(shape output)
-		(at 80.01 72.39 180)
-		(effects
-			(font
-				(size 1.27 1.27)
-			)
-			(justify right)
-		)
-	)
-	(hierarchical_label "MOTOR0_IN1"
-		(shape output)
-		(at 80.01 49.53 180)
-		(effects
-			(font
-				(size 1.27 1.27)
-			)
-			(justify right)
 		)
 	)
@@
 			)
 		)
-		(property "Value" "100u"
+		(property "Value" "120u"
 			(at 43.18 38.9381 0)
 			(effects
@@
 			)
 		)
-		(property "Footprint" "Capacitor_SMD:CP_Elec_6.3x7.7"
+		(property "Footprint" "Capacitor_SMD:CP_Elec_10x12.5"
 			(at 40.64 38.1 0)
 			(effects
@@
 			)
 		)
-		(property "LCSC" "C3338"
+		(property "LCSC" "C24725845"
 			(at 40.64 38.1 0)
 			(effects

Commit message: pcb
Parts:
- C3: footprint Capacitor_SMD:CP_Elec_10x12.5 -> Capacitor_SMD:CP_Elec_10x12.6
- J19, J4: now not fitted
- J2: LCSC C132132 -> (none)
Connections:
- net +5V: now also J2.3 (Pin_3)
- net ESC4: now also J4.12 (Pin_12); no longer J4.11 (Pin_11)
- net ESC5: now also J4.11 (Pin_11); no longer J4.12 (Pin_12)
- net GND: now also J2.10 (Pin_10), J2.13 (Pin_13), J2.19 (Pin_19), J2.26 (Pin_26), J2.29 (Pin_29), J2.33 (Pin_33), J2.40 (Pin_40)
- net PI_SCL: now also J19.14 (Pin_14), R12.2; no longer J19.15 (Pin_15), R13.2
- net PI_SDA: now also J19.15 (Pin_15), R13.2; no longer J19.14 (Pin_14), R12.2
- no-connect marks 48 -> 40
