File: LapisHAT/tooling.kicad_sch (KiCad schematic)
At the start: 40 parts, among them J10 Conn_01x02, J11 Conn_01x02, J12 Conn_01x02, J13 Conn_01x03, J14 Conn_01x03, J15 Conn_01x03, J16 Conn_01x03, J17 Conn_01x02, J18 Conn_01x02, J3 Conn_01x07, J4 Conn_01x07, J5 Conn_01x02, J6 Conn_01x02, J7 Conn_01x02, J8 Conn_01x02, J9 Conn_01x02, Q1 Q_NMOS_GSD, Q2 Q_NMOS_GSD, U1 NC7SZ18P6X, U2 NC7SZ18P6X, U3 NC7SZ18P6X, U4 DRV8231ADSG, U5 NC7SZ18P6X, U6 DRV8231ADSG

Commit message: Initial schematic
Parts:
- removed J3, J4: Conn_01x07, Connector_PinHeader_2.54mm:PinHeader_1x07_P2.54mm_Vertical, symbol Connector_Generic:Conn_01x07
- added C18, C21: 47u, Capacitor_SMD:C_0805_2012Metric, symbol Device:C_Small
- added C19, C20, C22, C23: 100n, Capacitor_SMD:C_0603_1608Metric, symbol Device:C_Small
- added J3, J4: Conn_01x06, Connector_PinHeader_2.54mm:PinHeader_1x06_P2.54mm_Vertical, symbol Connector_Generic:Conn_01x06
- added R7, R8: 10k, Resistor_SMD:R_0603_1608Metric, symbol Device:R_Small_US
- added U10, U11: DRV8231ADSG, Package_SON:WSON-8-1EP_2x2mm_P0.5mm_EP0.9x1.6mm, symbol Driver_Motor:DRV8231ADSG
Connections:
- net +12V: now also C18.1, C20.1, C21.1, C23.1, U10.5 (VM), U11.5 (VM)
- net +3V3: now also C19.1, C22.1, J3.1 (Pin_1), J4.1 (Pin_1), U10.4 (VREF), U11.4 (VREF)
- net ENCODER0_SCL: now also J3.5 (Pin_5)
- net ENCODER0_SDA: now also J3.4 (Pin_4)
- net ENCODER1_SCL: now also J4.5 (Pin_5)
- net ENCODER1_SDA: now also J4.4 (Pin_4)
- net GND: now also C18.2, C19.2, C20.2, C21.2, C22.2, C23.2, J3.6 (Pin_6), J4.6 (Pin_6), R7.2, R8.2, U10.7 (GND), U10.9 (GND), U11.7 (GND), U11.9 (GND)
- net MOTOR3_OUT1: now reaches J6.1 (Pin_1), U6.6 (OUT1)
- net MOTOR3_OUT2: now reaches J6.2 (Pin_2), U6.8 (OUT2)
- net at U1.6 (Y0): now also U11.3 (IN1)
- net at U1.4 (Y1): now also U11.2 (IN2)
- net MOTOR2_OUT1: now reaches J5.1 (Pin_1), U4.6 (OUT1)
- net MOTOR2_OUT2: now reaches J5.2 (Pin_2), U4.8 (OUT2)
- net at U2.4 (Y1): now also U10.2 (IN2)
- net at U2.6 (Y0): now also U10.3 (IN1)
- new net: R8.1, U11.1 (IPROPI)
- new net: R7.1, U10.1 (IPROPI)
- new net MOTOR0_OUT1: J3.2 (Pin_2), U11.6 (OUT1)
- new net MOTOR0_OUT2: J3.3 (Pin_3), U11.8 (OUT2)
- new net MOTOR1_OUT1: J4.2 (Pin_2), U10.6 (OUT1)
- new net MOTOR1_OUT2: J4.3 (Pin_3), U10.8 (OUT2)
Other:
- moved on the sheet: C1, C10, C11, C12, C13, C14, C2, C3, C4, C5, C6, C7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

Commit message: New Lapis Hat
Parts:
- removed C1, C19, C2, C20, C22, C23, C3, C7: 100n, Capacitor_SMD:C_0603_1608Metric, symbol Device:C_Small
- removed C18, C21: 47u, Capacitor_SMD:C_0805_2012Metric, symbol Device:C_Small
- removed J3, J4: Conn_01x06, Connector_PinHeader_2.54mm:PinHeader_1x06_P2.54mm_Vertical, symbol Connector_Generic:Conn_01x06
- removed R7, R8: 10k, Resistor_SMD:R_0603_1608Metric, symbol Device:R_Small_US
- removed U1, U2, U3, U5: NC7SZ18P6X, Package_TO_SOT_SMD:SOT-363_SC-70-6, symbol Lapis:NC7SZ18P6X
- removed U10, U11: DRV8231ADSG, Package_SON:WSON-8-1EP_2x2mm_P0.5mm_EP0.9x1.6mm, symbol Driver_Motor:DRV8231ADSG
- added C1, C2: 10u, Capacitor_SMD:CP_Elec_4x5.4, symbol Device:C_Polarized_Small_US
- added J3: Conn_01x02, footprints:Molex-43650-0227_-MFG, symbol Connector_Generic:Conn_01x02
- added R3, R4, R5, R6: 10k, Resistor_SMD:R_0603_1608Metric, symbol Device:R_Small_US
- J10, J11, J12, J7, J8, J9: footprint Connector_PinHeader_2.54mm:PinHeader_1x02_P2.54mm_Vertical -> Connector_Molex:Molex_SL_171971-0002_1x02_P2.54mm_Vertical; LCSC (none) -> C585468
- J13, J14, J15, J16: footprint Connector_PinSocket_2.54mm:PinSocket_1x03_P2.54mm_Vertical -> Connector_Molex:Molex_SL_171971-0003_1x03_P2.54mm_Vertical
- J17, J18, J5, J6: footprint Connector_PinHeader_2.54mm:PinHeader_1x02_P2.54mm_Vertical -> footprints:Molex-43650-0227_-MFG; LCSC (none) -> C585468
Connections:
- net MOTOR2_OUT1 is gone; now on net MOTOR0_OUT1: J5.1 (Pin_1), U4.6 (OUT1)
- net MOTOR2_OUT2 is gone; now on net MOTOR0_OUT2: J5.2 (Pin_2), U4.8 (OUT2)
- net MOTOR3_OUT1 is gone; now on net MOTOR0_OUT1: J6.1 (Pin_1), U6.6 (OUT1)
- net MOTOR3_OUT2 is gone; now on net MOTOR0_OUT2: J6.2 (Pin_2), U6.8 (OUT2)
- net +12V: now also C1.1, C2.1, J3.2 (Pin_2)
- net GND: now also C1.2, C2.2, J3.1 (Pin_1), R3.1, R4.1, R5.1, R6.1
- net MOTOR0_IN2: now reaches U4.2 (IN2)
- net MOTOR0_IN2: now also R4.2
- net MOTOR0_IN1: now reaches U4.3 (IN1)
- net MOTOR0_IN1: now also R3.2
- net MOTOR1_IN2: now reaches U6.2 (IN2)
- net MOTOR1_IN2: now also R6.2
- net MOTOR1_IN1: now reaches U6.3 (IN1)
- net MOTOR1_IN1: now also R5.2
Other:
- note removed: "Encoder/Camera Motor Headers"
- moved on the sheet: C10, C11, C12, C13, C14, C4, C5, C6, C8, C9, J10, J11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

Commit message: Set JLC part for connector
Parts:
- J13, J14, J15, J16: LCSC (none) -> C586606
Changed lines of the file:
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@@
 			)
 		)
-		(property "LCSC" ""
+		(property "LCSC" "C586606"
 			(at 182.88 72.39 0)
 			(effects
@@
 			)
 		)
-		(property "LCSC" ""
+		(property "LCSC" "C586606"
 			(at 182.88 95.25 0)
 			(effects
@@
 			)
 		)
-		(property "LCSC" ""
+		(property "LCSC" "C586606"
 			(at 213.36 95.25 0)
 			(effects
@@
 			)
 		)
-		(property "LCSC" ""
+		(property "LCSC" "C586606"
 			(at 213.36 72.39 0)
 			(effects

Commit message: Some review changes
Parts:
- C1, C2: value 10u -> 330u; LCSC C3343 -> C225873
- U4, U6: LCSC C5139865 -> C3681197
Connections:
- net GND: now also R1.1, R2.1, U4.1 (IPROPI), U6.1 (IPROPI); no longer R1.2, R2.2
- net LED0: now also R1.2
- net LED1: now also R2.2
- net MOTOR0_OUT1: no longer J6.1 (Pin_1), U6.6 (OUT1)
- net MOTOR0_OUT2: no longer J6.2 (Pin_2), U6.8 (OUT2)
- new net MOTOR1_OUT1: J6.1 (Pin_1), U6.6 (OUT1)
- new net MOTOR1_OUT2: J6.2 (Pin_2), U6.8 (OUT2)
Other:
- moved on the sheet: C2, J5, J6

Commit message: another layout
Parts:
- J10, J11, J12, J7, J8, J9: footprint Connector_Molex:Molex_SL_171971-0002_1x02_P2.54mm_Vertical -> footprints:CONN_70553-xxxx_02_MOL; LCSC C585468 -> C588446
- J3: footprint footprints:Molex-43650-0227_-MFG -> Connector_Molex:Molex_Micro-Fit_3.0_43650-0200_1x02_P3.00mm_Horizontal; LCSC C585468 -> C192562
Changed lines of the file:
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@@
 			)
 		)
-		(property "Footprint" "Connector_Molex:Molex_SL_171971-0002_1x02_P2.54mm_Vertical"
+		(property "Footprint" "footprints:CONN_70553-xxxx_02_MOL"
 			(at 142.24 67.31 0)
 			(effects
@@
 			)
 		)
-		(property "LCSC" "C585468"
+		(property "LCSC" "C588446"
 			(at 142.24 67.31 0)
 			(effects
@@
 			)
 		)
-		(property "Footprint" "Connector_Molex:Molex_SL_171971-0002_1x02_P2.54mm_Vertical"
+		(property "Footprint" "footprints:CONN_70553-xxxx_02_MOL"
 			(at 160.02 102.87 0)
 			(effects
@@
 			)
 		)
-		(property "LCSC" "C585468"
+		(property "LCSC" "C588446"
 			(at 160.02 102.87 0)
 			(effects
@@
 			)
 		)
-		(property "Footprint" "footprints:Molex-43650-0227_-MFG"
+		(property "Footprint" "Connector_Molex:Molex_Micro-Fit_3.0_43650-0200_1x02_P3.00mm_Horizontal"
 			(at 19.05 29.21 0)
 			(effects
@@
 			)
 		)
-		(property "LCSC" "C585468"
+		(property "LCSC" "C192562"
 			(at 19.05 29.21 0)
 			(effects
@@
 			)
 		)
-		(property "Footprint" "Connector_Molex:Molex_SL_171971-0002_1x02_P2.54mm_Vertical"
+		(property "Footprint" "footprints:CONN_70553-xxxx_02_MOL"
 			(at 142.24 85.09 0)
 			(effects
@@
 			)
 		)
-		(property "LCSC" "C585468"
+		(property "LCSC" "C588446"
 			(at 142.24 85.09 0)
 			(effects
@@
 			)
 		)
-		(property "Footprint" "Connector_Molex:Molex_SL_171971-0002_1x02_P2.54mm_Vertical"
+		(property "Footprint" "footprints:CONN_70553-xxxx_02_MOL"
 			(at 160.02 67.31 0)
 			(effects
@@
 			)
 		)
-		(property "LCSC" "C585468"
+		(property "LCSC" "C588446"
 			(at 160.02 67.31 0)
 			(effects
@@
 			)
 		)
-		(property "Footprint" "Connector_Molex:Molex_SL_171971-0002_1x02_P2.54mm_Vertical"
+		(property "Footprint" "footprints:CONN_70553-xxxx_02_MOL"
 			(at 160.02 85.09 0)
 			(effects
@@
 			)
 		)
-		(property "LCSC" "C585468"
+		(property "LCSC" "C588446"
 			(at 160.02 85.09 0)
 			(effects
@@
 			)
 		)
-		(property "Footprint" "Connector_Molex:Molex_SL_171971-0002_1x02_P2.54mm_Vertical"
+		(property "Footprint" "footprints:CONN_70553-xxxx_02_MOL"
 			(at 142.24 102.87 0)
 			(effects
@@
 			)
 		)
-		(property "LCSC" "C585468"
+		(property "LCSC" "C588446"
 			(at 142.24 102.87 0)
 			(effects

Commit message: pcb
Parts:
- removed C11, C12, C13, C14: 100u, Capacitor_SMD:CP_Elec_6.3x7.7, symbol Device:C_Polarized_Small_US
- removed C2: 330u, Capacitor_SMD:CP_Elec_4x5.4, symbol Device:C_Polarized_Small_US
- added R10, R11: 10k, Resistor_SMD:R_0603_1608Metric, symbol Device:R_Small_US
- C1: value 330u -> 120u; footprint Capacitor_SMD:CP_Elec_4x5.4 -> Capacitor_SMD:CP_Elec_10x12.6; LCSC C225873 -> C24725845
- C5, C8: footprint Capacitor_SMD:C_0805_2012Metric -> Capacitor_SMD:C_1206_3216Metric; LCSC C16780 -> C403725
- J17, J18, J5, J6: footprint footprints:Molex-43650-0227_-MFG -> Connector_Molex:Molex_Micro-Fit_3.0_43650-0200_1x02_P3.00mm_Horizontal; LCSC C585468 -> C192562
- U4, U6: LCSC C3681197 -> C5139865
Connections:
- net GND: now also R10.2, R11.2; no longer U4.1 (IPROPI), U6.1 (IPROPI)
- net MOTOR0_OUT1: now also J5.2 (Pin_2); no longer J5.1 (Pin_1)
- net MOTOR0_OUT2: now also J5.1 (Pin_1); no longer J5.2 (Pin_2)
- net MOTOR1_OUT1: now also J6.2 (Pin_2); no longer J6.1 (Pin_1)
- net MOTOR1_OUT2: now also J6.1 (Pin_1); no longer J6.2 (Pin_2)
- net LED0_PIN: now reaches J17.2 (Pin_2), Q1.3 (D)
- net LED1_PIN: now reaches J18.2 (Pin_2), Q2.3 (D)
- new net: R10.1, U6.1 (IPROPI)
- new net: R11.1, U4.1 (IPROPI)
Other:
- moved on the sheet: J18, J6
